File: STAGE_POWER.kicad_sch (KiCad schematic)
At the start: 6 parts, among them Q1 2SC5200, Q2 2SA1943

Commit message: mejorando pistas
Parts:
- Q10: renamed from Q2; LCSC Part (none) -> C480004; Manufacturer (none) -> Toshiba Semiconductor and Storage; Mfr. Part (none) -> 2SA1943-O(Q); Price (none) -> 2.84
- Q9: renamed from Q1; LCSC Part (none) -> C2920870; Manufacturer (none) -> onsemi; Mfr. Part (none) -> 2SC5200OTU; Price (none) -> 4.99
- R17: renamed from R1; symbol Device:R -> Device:R_US
- R18: renamed from R2; symbol Device:R -> Device:R_US
- R19: renamed from R3; symbol Device:R -> Device:R_US
- R20: renamed from R4; value 2.2 -> 0.22; symbol Device:R -> Device:R_US
